File: kicad/current_version/working/working.kicad_pcb (KiCad board)
At the start: 2 copper layers, 3 parts

Commit message: commiting after auto generation
Other:
- board outline added: 65 x 80 mm
Changed lines of the file:
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@@
     )
   )
+  (gr_line (start 30 30) (end 35 30)
+    (stroke (width 0.1) (type default)) (layer "Edge.Cuts"))
+  (gr_line (start 30 110) (end 30 30)
+    (stroke (width 0.1) (type default)) (layer "Edge.Cuts"))
+  (gr_line (start 95 30) (end 95 110)
+    (stroke (width 0.1) (type default)) (layer "Edge.Cuts"))
+  (gr_line (start 40 110) (end 30 110)
+    (stroke (width 0.1) (type default)) (layer "Edge.Cuts"))
+  (gr_line (start 35 30) (end 95 30)
+    (stroke (width 0.1) (type default)) (layer "Edge.Cuts"))
+  (gr_line (start 95 110) (end 40 110)
+    (stroke (width 0.1) (type default)) (layer "Edge.Cuts"))
   (segment (start 53.42 48.18) (end 53.42 46.50312) (width 0.25) (layer "B.Cu") (net 1))
   (segment (start 52.07 49.53) (end 53.42 48.18) (width 0.25) (layer "B.Cu") (net 1))
